File: Hardware/GuitarPedal125b/pcb/Audio_Input_Buffer.kicad_sch (KiCad schematic)
At the start: 11 parts, among them U2 MCP6004

Commit message: Replace screen and encoder by 3 toggle switches and SD card reader.
Parts:
- C5, C6: MPN (none) -> C49678
- C7, C8: MPN (none) -> C15850
- R1, R2, R4, R5: MPN (none) -> C26112
- R3, R6: MPN (none) -> C149504
- U2: MPN (none) -> C7378
