File: Hardware/GuitarPedal125b/pcb/Audio_Output_Buffer.kicad_sch (KiCad schematic)
At the start: 19 parts, among them U3 OPA1652AID

Commit message: Replace screen and encoder by 3 toggle switches and SD card reader.
Parts:
- C10, C9: MPN (none) -> C28260
- C11, C12, C15, C16: MPN (none) -> C15850
- C13, C14: MPN (none) -> C49678
- R10, R11, R12, R15, R16, R9: MPN (none) -> C26112
- R13, R14: MPN (none) -> C17408
- R7, R8: MPN (none) -> C26010
- U3: MPN (none) -> C30025
