File: Hardware/GuitarPedal125b/pcb/Audio_True_Bypass_Stereo.kicad_sch (KiCad schematic)
At the start: 10 parts, among them K1 G6K-2, K2 G6K-2, Q1 SS8050, U5 CPC1018N, U6 CPC1018N

Commit message: Replace screen and encoder by 3 toggle switches and SD card reader.
Parts:
- D3, D4: MPN (none) -> C108803
- K1, K2: MPN (none) -> C397140
- Q1: MPN (none) -> C2150
- R21, R22, R23: MPN (none) -> C17513
- U5, U6: MPN (none) -> C133069
