File: Hardware/GuitarPedal125b/pcb/Midi_InOut.kicad_sch (KiCad schematic)
At the start: 7 parts, among them U4 H11L1

Commit message: Replace screen and encoder by 3 toggle switches and SD card reader.
Parts:
- C17: MPN (none) -> C49678
- D2: MPN (none) -> C81598
- R17: MPN (none) -> C17557
- R18: MPN (none) -> C17415
- R19: MPN (none) -> C17634
- R20: MPN (none) -> C17710
- U4: MPN (none) -> C78589
