File: Hardware/GuitarPedal125b/pcb/Power.kicad_sch (KiCad schematic)
At the start: 6 parts, among them U1 LD1117S50TR_SOT223

Commit message: Replace screen and encoder by 3 toggle switches and SD card reader.
Parts:
- C1, C4: MPN (none) -> C15850
- C2, C3: MPN (none) -> C49678
- D1: MPN (none) -> C727113
- U1: MPN (none) -> C81157
